File: ams_measurement.kicad_pcb (KiCad board)
At the start: 2 copper layers, 360.5 x 16 mm, 29 parts, among them J1 S1961-46R, J10 S1961-46R, J11 S1961-46R, J12 Conn_02x10_Odd_Even, J2 S1961-46R, J3 S1961-46R, J4 S1961-46R, J5 S1961-46R, J6 S1961-46R, J7 S1961-46R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

Commit message: Changed connector to TE 5-5530843-0
Parts:
- J12: footprint Connector_IDC:IDC-Header_2x10_P2.54mm_Vertical -> Connector_PCBEdge:555308430
- moved J12 1.00 mm to (221.7, 151.5), turned to 180 degrees
Routing:
- net /TH3+: track 23.9 -> 26.3 mm
- net /C8+: track 30.1 -> 28.1 mm
- net /TH2-: track 130.2 -> 129.1 mm
- net /TH1+: track 84.8 -> 84.0 mm
- net /C10+: track 143.4 -> 144.0 mm
- net /C5+: track 143.9 -> 144.4 mm
- net /TH3-: track 22.4 -> 21.9 mm

Commit message: Revert "Changed connector to TE 5-5530843-0"
Parts:
- J12: footprint Connector_PCBEdge:555308430 -> Connector_IDC:IDC-Header_2x10_P2.54mm_Vertical
- moved J12 1.00 mm to (221.7, 152.5), turned to -90 degrees
Routing:
- net /TH3+: track 26.3 -> 23.9 mm
- net /C8+: track 28.1 -> 30.1 mm
- net /TH2-: track 129.1 -> 130.2 mm
- net /TH1+: track 84.0 -> 84.8 mm
- net /C10+: track 144.0 -> 143.4 mm
- net /C5+: track 144.4 -> 143.9 mm
- net /TH3-: track 21.9 -> 22.4 mm
