File: ams_measurement.kicad_sch (KiCad schematic)
At the start: 26 parts, among them J1 S1961-46R, J10 S1961-46R, J11 S1961-46R, J12 Conn_02x10_Odd_Even, J2 S1961-46R, J3 S1961-46R, J4 S1961-46R, J5 S1961-46R, J6 S1961-46R, J7 S1961-46R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

Commit message: Changed connector to TE 5-5530843-0
Parts:
- J12: footprint Connector_IDC:IDC-Header_2x10_P2.54mm_Vertical -> Connector_PCBEdge:555308430
Changed lines of the file:
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@@
       (effects (font (size 1.27 1.27)))
     )
-    (property "Footprint" "Connector_IDC:IDC-Header_2x10_P2.54mm_Vertical" (at 189.23 59.69 0)
+    (property "Footprint" "Connector_PCBEdge:555308430" (at 189.23 59.69 0)
       (effects (font (size 1.27 1.27)) hide)
     )

Commit message: Revert "Changed connector to TE 5-5530843-0"
Parts:
- J12: footprint Connector_PCBEdge:555308430 -> Connector_IDC:IDC-Header_2x10_P2.54mm_Vertical
Changed lines of the file:
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@@
       (effects (font (size 1.27 1.27)))
     )
-    (property "Footprint" "Connector_PCBEdge:555308430" (at 189.23 59.69 0)
+    (property "Footprint" "Connector_IDC:IDC-Header_2x10_P2.54mm_Vertical" (at 189.23 59.69 0)
       (effects (font (size 1.27 1.27)) hide)
     )
