File: PUTM_EV_BMS_HV_MEASUREMENT_2024/ams_measurement.kicad_pcb (KiCad board)
At the start: 2 copper layers, 345 x 19.4 mm, 30 parts, among them J1 CELL_PAD, J10 CELL_PAD, J11 CELL_PAD, J12 Conn_02x10_Odd_Even, J2 CELL_PAD, J3 CELL_PAD, J4 CELL_PAD, J5 CELL_PAD, J6 CELL_PAD, J7 CELL_PAD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

Commit message: Changed thermistor position
Parts:
- moved TH4 235.7 mm to (147.8, 150.2)
- moved TH1 148.7 mm to (383.2, 150.5)
- moved J6 8.00 mm to (51.8, 150.0)
- moved F6 7.16 mm to (70.9, 150.5)
- moved TH2 7.07 mm to (49.5, 157.5)
- moved F4 3.25 mm to (181.6, 150.5)
- moved J4 3.25 mm to (172.2, 150.0)
Routing:
- net /TH1+: track 18.7 -> 167.5 mm
- net /TH1-: track 23.9 -> 172.7 mm
- net /TH4-: track 179.4 -> 63.2 mm
- net /TH4+: track 174.1 -> 65.7 mm
- net /C3+: track 21.2 -> 17.9 mm
- net /C4+: track 74.7 -> 77.9 mm
- net /TH2+: track 158.0 -> 160.8 mm, vias 0 -> 2
- net /C5+: track 125.7 -> 127.2 mm
- net Net-(F6-Pad1): track 18.8 -> 17.5 mm

Commit message: Wider tracks, vias and common -
Tracks now 1.2mm
Vias added to WAGO connector footprint
All thermistors now have common negative pin
Changes to thermistor placement (added TH5)
Parts:
- added TH5: TT7-10KC8-3, Connector_PinHeader_2.54mm:PinHeader_1x02_P2.54mm_Vertical, F.Cu at (276.2, 157.5)
- moved TH2 187.6 mm to (237.0, 150.5)
- moved TH3 112.2 mm to (70.7, 150.5)
- moved TH4 26.3 mm to (122.5, 157.5)
- moved J6 8.46 mm to (54.5, 158.0)
- moved F6 7.22 mm to (69.1, 157.5)
- moved F9 2.49 mm to (239.6, 157.8)
- moved J9 2.48 mm to (249.0, 158.0)
- moved J4 2.27 mm to (170.0, 150.0)
- moved F4 2.27 mm to (179.4, 150.5)
- moved F3 1.73 mm to (255.4, 150.5)
- moved J3 1.73 mm to (264.7, 150.0)
- moved F1 0.25 mm to (351.4, 150.2)
- moved F10 0.25 mm to (294.9, 157.8)
- moved F2 0.25 mm to (308.5, 150.2)
- moved F7 0.25 mm to (106.4, 157.8)
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Connections:
- J12 pad 10: /TH4- -> /TH5+
- J12 pad 11: /TH3+ -> /TH-
- J12 pad 12: /TH3- -> /TH-
- J12 pad 13: /TH2+ -> unconnected-(J12-Pin_13-Pad13)
- J12 pad 14: /TH2- -> /TH4+
- J12 pad 15: unconnected-(J12-Pin_15-Pad15) -> /TH3+
- J12 pad 6: /TH1- -> unconnected-(J12-Pin_6-Pad6)
- J12 pad 9: /TH4+ -> /TH2+
- TH1 pad 2: /TH1- -> /TH-
- TH2 pad 2: /TH2- -> /TH-
- TH3 pad 2: /TH3- -> /TH-
- TH4 pad 2: /TH4- -> /TH-
Routing:
- net /TH-: track 0.00 -> 330.9 mm
- net /TH1-: track 172.7 -> 0.00 mm
- net /TH2-: track 155.4 -> 0.00 mm
- net /TH2+: track 160.8 -> 26.3 mm
- net /TH3+: track 30.8 -> 139.1 mm, vias 1 -> 0
- net /TH5+: track 0.00 -> 69.6 mm
- net /TH4-: track 63.2 -> 0.00 mm
- net Net-(F2-Pad1): track 7.38 -> 42.4 mm, vias 0 -> 18
- net Net-(F10-Pad1): track 7.97 -> 39.2 mm, vias 0 -> 18
- net Net-(F8-Pad1): track 7.32 -> 36.6 mm, vias 0 -> 18
- net Net-(F1-Pad1): track 13.0 -> 39.9 mm, vias 0 -> 18
- net Net-(F7-Pad1): track 7.33 -> 33.5 mm, vias 0 -> 18
- net Net-(F9-Pad1): track 7.71 -> 33.8 mm, vias 0 -> 18
- net Net-(F11-Pad1): track 7.71 -> 33.7 mm, vias 0 -> 18
- net Net-(F3-Pad1): track 7.27 -> 32.4 mm, vias 0 -> 18
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- added copper zone on B.Cu, net Net-(F1-Pad1)
- added copper zone on B.Cu, net Net-(F10-Pad1)
- added copper zone on B.Cu, net Net-(F11-Pad1)
- added copper zone on B.Cu, net Net-(F2-Pad1)
- added copper zone on B.Cu, net Net-(F3-Pad1)
- added copper zone on B.Cu, net Net-(F4-Pad1)
- added copper zone on B.Cu, net Net-(F5-Pad1)
- added copper zone on B.Cu, net Net-(F6-Pad1)
- added copper zone on B.Cu, net Net-(F7-Pad1)
- added copper zone on B.Cu, net Net-(F8-Pad1)
- added copper zone on B.Cu, net Net-(F9-Pad1)

Commit message: Preparation for production
Parts:
- moved REF** 1.50 mm to (358.0, 154.0)
- moved F1 1.25 mm to (350.1, 150.2)
- moved F10 1.25 mm to (293.6, 157.8)
- moved F11 1.25 mm to (365.9, 157.5)
- moved F2 1.25 mm to (307.2, 150.2)
- moved F3 1.25 mm to (254.1, 150.5)
- moved F4 1.25 mm to (178.1, 150.5)
- moved F5 1.25 mm to (121.1, 150.5)
- moved F6 1.25 mm to (67.9, 157.5)
- moved F7 1.25 mm to (105.1, 157.8)
- moved F8 1.25 mm to (162.1, 157.8)
- moved F9 1.25 mm to (238.4, 157.8)
- moved G*** 1.25 mm to (134.8, 154.0)
- moved J1 1.25 mm to (365.2, 150.0)
- moved J10 1.25 mm to (303.2, 158.0)
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Routing:
- net Net-(F1-Pad1): track 39.9 -> 35.6 mm
- net Net-(F6-Pad1): track 40.2 -> 43.5 mm
- net Net-(F2-Pad1): track 42.4 -> 45.6 mm
- net Net-(F5-Pad1): track 30.9 -> 28.9 mm
- net Net-(F4-Pad1): track 31.8 -> 29.9 mm
- net Net-(F11-Pad1): track 33.7 -> 32.3 mm
- net Net-(F3-Pad1): track 32.4 -> 31.2 mm
- net Net-(F7-Pad1): track 33.5 -> 32.3 mm
- net /TH3+: track 139.1 -> 139.7 mm
- net Net-(F8-Pad1): track 36.6 -> 36.1 mm

Commit message: Board dimensions changed
Parts:
- moved F1 1.01 mm to (350.0, 151.3)
- moved J6 0.87 mm to (52.4, 158.2)
- moved F8 0.76 mm to (162.0, 157.0)
- moved J5 0.75 mm to (111.7, 150.8)
- moved J4 0.75 mm to (168.7, 150.8)
- moved F2 0.75 mm to (307.2, 151.0)
- moved J10 0.75 mm to (303.2, 157.2)
- moved F7 0.75 mm to (105.1, 157.0)
- moved F9 0.75 mm to (238.4, 157.0)
- moved F10 0.75 mm to (293.6, 157.0)
- moved J9 0.75 mm to (247.8, 157.2)
- moved J11 0.75 mm to (375.0, 157.2)
- moved F6 0.71 mm to (68.4, 157.0)
- moved F5 0.58 mm to (120.8, 151.0)
- moved F4 0.57 mm to (177.8, 151.0)
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Routing:
- net Net-(F8-Pad1): track 36.1 -> 7.37 mm
- net Net-(F4-Pad1): track 29.9 -> 7.37 mm
- net Net-(F2-Pad1): track 45.6 -> 24.1 mm
- net /TH-: track 330.9 -> 348.2 mm, vias 0 -> 1
- net Net-(F6-Pad1): track 43.5 -> 27.2 mm
- net Net-(F9-Pad1): track 33.6 -> 21.3 mm
- net Net-(F11-Pad1): track 32.3 -> 20.3 mm
- net Net-(F7-Pad1): track 32.3 -> 20.6 mm
- net Net-(F10-Pad1): track 39.2 -> 28.2 mm
- net Net-(F3-Pad1): track 31.2 -> 20.5 mm
- net Net-(F1-Pad1): track 35.6 -> 26.5 mm
- net Net-(F5-Pad1): track 28.9 -> 20.3 mm
- net /TH3+: track 139.7 -> 136.0 mm, vias 0 -> 3
- net /C6+: track 94.9 -> 97.2 mm, vias 1 -> 0
- net /TH5+: track 69.6 -> 67.6 mm
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Other:
- board size 345 x 19.4 mm -> 345 x 24 mm
